File: clocky.kicad_sch (KiCad schematic)
At the start: 78 parts, among them J1 Bot 50 pin, J2 Bot 40 pin, J3 Top 50 pin, J4 Top 40 pin, J5 Power, J6 JST_PH, J8 Program, Q1 AO3401A, U1 HEF4094B, U10 TMP117xxDRV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

Commit message: Final updates.  Ordered.
Parts:
- added R20: 10k, Resistor_SMD:R_0603_1608Metric, symbol Device:R
- C9: footprint Capacitor_SMD:C_0402_1005Metric -> Capacitor_SMD:C_0603_1608Metric; JLCPCB C63949 -> (none); now left out of the parts list
- D2, D6, J5, R18, R19: now left out of the parts list
- Q1: value AO3401A -> SI2301A; JLCPCB C15127 -> C10487
- R5: now in the parts list
- U7: footprint Package_SON:Texas_S-PWSON-N10_ThermalVias -> Package_SON:Texas_S-PWSON-N10
- renumbered R20 to R21
Connections:
- net +3V3: now also R20.2
- net Alert: now also R20.1
- net Minus: now also R10.2, U9.29 (PA8); no longer R11.2, U9.31 (PA10)
- net MinusPad: now also R10.1, TP1.1; no longer R11.1, TP2.1
- net Plus: now also R11.2, U9.31 (PA10); no longer R10.2, U9.29 (PA8)
- net PlusPad: now also R11.1, TP2.1; no longer R10.1, TP1.1
Changed lines of the file:
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@@
 	)
 	(junction
-		(at 92.71 38.1)
-		(diameter 0)
-		(color 0 0 0 0)
-	)
-	(junction
 		(at 50.8 30.48)
 		(diameter 0)
@@
 	)
 	(junction
+		(at 248.92 40.64)
+		(diameter 0)
+		(color 0 0 0 0)
+	)
+	(junction
 		(at 44.45 78.74)
 		(diameter 0)
@@
 	)
 	(junction
+		(at 248.92 30.48)
+		(diameter 0)
+		(color 0 0 0 0)
+	)
+	(junction
 		(at 137.16 69.85)
 		(diameter 0)
@@
 	(wire
 		(pts
+			(xy 248.92 40.64) (xy 261.62 40.64)
+		)
+		(stroke
+			(width 0)
+			(type default)
+		)
+	)
+	(wire
+		(pts
 			(xy 146.05 53.34) (xy 146.05 58.42)
 		)
@@
 	(wire
 		(pts
-			(xy 50.8 68.58) (xy 50.8 71.12)
-		)
-		(stroke
-			(width 0)
-			(type default)
-		)
-	)
-	(wire
-		(pts
 			(xy 259.08 128.27) (xy 254 128.27)
 		)
@@
 	(wire
 		(pts
-			(xy 247.65 40.64) (xy 261.62 40.64)
+			(xy 247.65 40.64) (xy 248.92 40.64)
 		)
 		(stroke
@@
 	(wire
 		(pts
+			(xy 248.92 30.48) (xy 237.49 30.48)
+		)
+		(stroke
+			(width 0)
+			(type default)
+		)
+	)
+	(wire
+		(pts
 			(xy 215.9 43.18) (xy 223.52 43.18)
 		)
@@
 	(wire
 		(pts
+			(xy 248.92 30.48) (xy 248.92 31.75)
+		)
+		(stroke
+			(width 0)
+			(type default)
+		)
+	)
+	(wire
+		(pts
 			(xy 119.38 157.48) (xy 132.08 157.48)
 		)
@@
 	(wire
 		(pts
-			(xy 251.46 30.48) (xy 237.49 30.48)
+			(xy 251.46 30.48) (xy 248.92 30.48)
 		)
 		(stroke
@@
 	(wire
 		(pts
-			(xy 92.71 38.1) (xy 91.44 38.1)
-		)
-		(stroke
-			(width 0)
-			(type default)
-		)
-	)
-	(wire
-		(pts
 			(xy 227.33 111.76) (xy 232.41 111.76)
 		)
@@
 	(wire
 		(pts
+			(xy 248.92 39.37) (xy 248.92 40.64)
+		)
+		(stroke
+			(width 0)
+			(type default)
+		)
+	)
+	(wire
+		(pts
 			(xy 153.67 80.01) (xy 157.48 80.01)
 		)
@@
 	)
 	(label "PlusPad"
-		(at 204.47 154.94 90)
+		(at 209.55 154.94 90)
 		(effects
 			(font
@@
 	)
 	(label "Plus"
-		(at 88.9 129.54 180)
+		(at 88.9 134.62 180)
 		(effects
 			(font
@@
 	)
 	(label "Minus"
-		(at 88.9 134.62 180)
+		(at 88.9 129.54 180)
 		(effects
 			(font
@@
 	)
 	(label "MinusPad"
-		(at 209.55 154.94 90)
+		(at 204.47 154.94 90)
 		(effects
 			(font
@@
 	)
 	(label "Minus"
-		(at 209.55 129.54 270)
+		(at 204.47 129.54 270)
 		(effects
 			(font
@@
 	)
 	(label "Plus"
-		(at 204.47 129.54 270)
+		(at 209.55 129.54 270)
 		(effects
 			(font
@@
 		(unit 1)
 		(exclude_from_sim no)
-		(in_bom no)
+		(in_bom yes)
 		(on_board yes)
 		(dnp no)
@@
 		(unit 1)
 		(exclude_from_sim no)
-		(in_bom yes)
+		(in_bom no)
 		(on_board yes)
 		(dnp yes)
@@
 			)
 		)
-		(property "Value" "AO3401A"
+		(property "Value" "SI2301A"
 			(at 114.3 39.37 90)
 			(effects
@@
 			)
 		)
-		(property "Datasheet" "http://www.aosmd.com/pdfs/datasheet/AO3401A.pdf"
+		(property "Datasheet" ""
 			(at 109.22 27.94 0)
 			(effects
@@
 			)
 		)
-		(property "Description" "-4.0A Id, -30V Vds, P-Channel MOSFET, SOT-23"
+		(property "Description" "P-Channel MOSFET, SOT-23"
 			(at 105.41 33.02 0)
 			(effects
@@
 			)
 		)
-		(property "JLCPCB" "C15127"
+		(property "JLCPCB" "C10487"
 			(at 105.41 33.02 0)
 			(effects
@@
 		(unit 1)
 		(exclude_from_sim no)
-		(in_bom yes)
+		(in_bom no)
 		(on_board yes)
 		(dnp yes)
@@
 	)
 	(symbol
+		(lib_id "Device:R")
+		(at 248.92 35.56 180)
+		(unit 1)
+		(exclude_from_sim no)
+		(in_bom no)
+		(on_board yes)
+		(dnp yes)
+		(property "Reference" "R20"
+			(at 246.888 35.56 90)
+			(effects
+				(font
+					(size 1.27 1.27)
+				)
+			)
+		)
+		(property "Value" "10k"
+			(at 248.92 35.56 90)
+			(effects
+				(font
+					(size 1.27 1.27)
+				)
+			)
+		)
+		(property "Footprint" "Resistor_SMD:R_0603_1608Metric"
+			(at 250.698 35.56 90)
+			(effects
+				(font
+					(size 1.27 1.27)
+				)
+				(hide yes)
+			)
+		)
+		(property "Datasheet" "~"
+			(at 248.92 35.56 0)
+			(effects
+				(font
+					(size 1.27 1.27)
+				)
+				(hide yes)
+			)
+		)
+		(property "Description" "Resistor"
+			(at 248.92 35.56 0)
+			(effects
+				(font
+					(size 1.27 1.27)
+				)
+				(hide yes)
+			)
+		)
+		(pin "1"
+		)
+		(pin "2"
+		)
+		(instances
+			(project "clocky"
+				(path "/1a152c6d-723d-49c0-9a40-41d8f1ee1a82"
+					(reference "R20")
+					(unit 1)
+				)
+			)
+		)
+	)
+	(symbol
 		(lib_id "Connector:Conn_01x25_Socket")
 		(at 160.02 115.57 90)
@@
 		(unit 1)
 		(exclude_from_sim no)
-		(in_bom yes)
+		(in_bom no)
 		(on_board yes)
 		(dnp no)
@@
 			)
 		)
-		(property "Footprint" "Capacitor_SMD:C_0402_1005Metric"
+		(property "Footprint" "Capacitor_SMD:C_0603_1608Metric"
 			(at 79.0448 38.1 0)
 			(effects
@@
 			)
 		)
-		(property "JLCPCB" "C63949"
+		(property "JLCPCB" ""
 			(at 80.01 41.91 0)
 			(effects
@@
 		(unit 1)
 		(exclude_from_sim no)
-		(in_bom yes)
+		(in_bom no)
 		(on_board yes)
 		(dnp yes)
@@
 		(unit 1)
 		(exclude_from_sim no)
-		(in_bom yes)
+		(in_bom no)
 		(on_board yes)
 		(dnp no)
@@
 		(unit 1)
 		(exclude_from_sim no)
-		(in_bom yes)
+		(in_bom no)
 		(on_board yes)
 		(dnp yes)
@@
 			)
 		)
-		(property "Footprint" "Package_SON:Texas_S-PWSON-N10_ThermalVias"
+		(property "Footprint" "Package_SON:Texas_S-PWSON-N10"
 			(at 64.77 57.15 0)
 			(effects
@@
 		(on_board yes)
 		(dnp yes)
-		(property "Reference" "R20"
+		(property "Reference" "R21"
 			(at 106.68 64.008 90)
 			(effects
@@
 			(project ""
 				(path "/1a152c6d-723d-49c0-9a40-41d8f1ee1a82"
-					(reference "R20")
+					(reference "R21")
 					(unit 1)
 				)
