File: monitor.kicad_sch (KiCad schematic)
At the start: 81 parts, among them J1 USB_C_Plug, J2 USB_C_Receptacle_USB2.0_14P, J3 Display, J4 Program, U1 STM32U031K8Ux, U201 OPA2388, U251 LM27761, U301 TPSM365R6V3RDNR, U401 TMP117xxDRV, U411 REF5025ADGK, U421 FXLS8971CF, Y1 32768Hz

Commit message: Board layout updated.
Parts:
- added C91, C92, C93, C94: 0u1, Capacitor_SMD:C_0402_1005Metric, symbol Device:C
- added D3: 1N5819, Diode_SMD:D_SOD-323, symbol Diode:1N5819WS
- added R42: 510k, Resistor_SMD:R_0402_1005Metric, symbol Device:R
- added R43: 10, Resistor_SMD:R_0402_1005Metric, symbol Device:R
- added R9: 10, Resistor_SMD:R_0603_1608Metric, symbol Device:R
- C1: renamed from C201; JLCPCB (none) -> C52923
- C2: renamed from C202; JLCPCB (none) -> C52923
- C3: renamed from C203; JLCPCB (none) -> C52923
- C41: renamed from C251; JLCPCB (none) -> C23733
- C43: renamed from C253; JLCPCB (none) -> C23733
- C44: renamed from C254; JLCPCB (none) -> C23733
- C51: JLCPCB (none) -> C52923
- C52: JLCPCB (none) -> C23733
- R1: renamed from R4; now left out of the parts list
- R2: renamed from R201; JLCPCB (none) -> C11702
- R41: renamed from R251; value ?? -> 200k; footprint Resistor_SMD:R_0603_1608Metric -> Resistor_SMD:R_0402_1005Metric; JLCPCB (none) -> C25764
- R5: renamed from R204; JLCPCB (none) -> C23153
- R6: renamed from R205; JLCPCB (none) -> C23153
- TP1, TP2, TP3, TP301: now left out of the parts list
- TP31: renamed from TP302; now left out of the parts list
- U2: renamed from U201; JLCPCB (none) -> C2059281; now left out of the parts list
- U4: renamed from U251; JLCPCB (none) -> C129351
- U5: renamed from U411; now left out of the parts list
- U6: renamed from U401; now left out of the parts list
- U7: renamed from U421; Height 1.3 -> (none); JLCPCB (none) -> C24123558; Manufacturer_Name NXP -> (none); Manufacturer_Part_Number FXLS8971CF -> (none)
- renumbered C9 to C11, C10 to C12, C11 to C13, C12 to C14, C13 to C16, C14 to C17, C301 to C31, C302 to C32, C303 to C33, C304 to C34, C305 to C35, C204 to C4, C252 to C42, C205 to C5, C411 to C53, C412 to C54, C413 to C55, C414 to C56, C15 to C57, C421 to C58, C20 to C61, D51 to D2, R7 to R11, R6 to R12, R202 to R3, R301 to R31, R203 to R4, R411 to R55, R401 to R56, R402 to R57, R403 to R58, R8 to R61, R9 to R62, R10 to R63, R11 to R64, R12 to R65, R5 to R66, R206 to R7, R207 to R8, U301 to U3
Connections:
- net GND: now also D3.2 (A), R42.2
- net ISense: now also R9.1; no longer U1.15 (PB1)
- net MGnd: now also C91.1, C92.1, C93.1, C94.1
- net UGnd: now also C91.2, C92.2, C93.2, C94.2
- net VSense1: now also C51.1, D2.1 (A), R51.2, R52.2
- net A2-: now reaches C3.2, R6.1, R8.1, U2.6 (-)
- net at R41.2, U4.5 (VFB): now also R42.1
- net A2+: now reaches C2.1, R4.2, R5.1, R7.1, U2.5 (+)
- net A1: now reaches C1.1, R3.2, R5.2, U2.1
- net A1-: now reaches C1.2, R2.1, R3.1, U2.2 (-)
- net -1V65 renamed -1V7
- net -1V7: now also R43.1; no longer C5.2, U2.4 (V-)
- new net -1V7F: C5.2, R43.2, U2.4 (V-)
- new net ISenseP: D3.1 (K), R9.2, U1.15 (PB1)
Other:
- moved on the sheet: C1, C2, C3, C57, H1, H2, H3, H4, R3, R4, R5, R56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

Commit message: Tweaks.  Fabbing.
Parts:
- D2: JLCPCB C2128 -> C68978
- R2: JLCPCB C11702 -> C21190
- R43: JLCPCB (none) -> C25077
- R51: JLCPCB (none) -> C22961
- R52: JLCPCB (none) -> C25803
- R53: JLCPCB (none) -> C23137
- R54: JLCPCB (none) -> C31850
- R8: JLCPCB C25083 -> C25803
- R9: footprint Resistor_SMD:R_0603_1608Metric -> Resistor_SMD:R_0402_1005Metric; JLCPCB (none) -> C25077; now in the parts list
Changed lines of the file:
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@@
 			)
 		)
-		(property "JLCPCB" "C25083"
+		(property "JLCPCB" "C25803"
 			(at 186.69 62.23 0)
 			(effects
@@
 			)
 		)
-		(property "JLCPCB" "C2128"
+		(property "JLCPCB" "C68978"
 			(at 119.38 59.69 0)
 			(effects
@@
 		(unit 1)
 		(exclude_from_sim no)
-		(in_bom no)
+		(in_bom yes)
 		(on_board yes)
 		(dnp no)
@@
 			)
 		)
-		(property "Footprint" "Resistor_SMD:R_0603_1608Metric"
+		(property "Footprint" "Resistor_SMD:R_0402_1005Metric"
 			(at 198.12 51.562 90)
 			(effects
@@
 			)
 		)
-		(property "JLCPCB" ""
+		(property "JLCPCB" "C25077"
 			(at 198.12 53.34 0)
 			(effects
@@
 			)
 		)
-		(property "JLCPCB" ""
+		(property "JLCPCB" "C25077"
 			(at 219.71 66.04 0)
 			(effects
@@
 			)
 		)
-		(property "JLCPCB" ""
+		(property "JLCPCB" "C25803"
 			(at 111.76 66.04 0)
 			(effects
@@
 			)
 		)
-		(property "JLCPCB" ""
+		(property "JLCPCB" "C31850"
 			(at 127 66.04 0)
 			(effects
@@
 			)
 		)
-		(property "JLCPCB" "C11702"
+		(property "JLCPCB" "C21190"
 			(at 146.05 53.34 0)
 			(effects
@@
 			)
 		)
-		(property "JLCPCB" ""
+		(property "JLCPCB" "C23137"
 			(at 127 54.61 0)
 			(effects
@@
 			)
 		)
-		(property "JLCPCB" ""
+		(property "JLCPCB" "C22961"
 			(at 111.76 54.61 0)
 			(effects

Commit message: Update the python scripts.
Parts:
- R3: JLCPCB C25083 -> C25803
Changed lines of the file:
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@@
 			)
 		)
-		(property "JLCPCB" "C25083"
+		(property "JLCPCB" "C25803"
 			(at 158.75 59.69 0)
 			(effects
